File: MCU Data Logger.kicad_sch (KiCad schematic)
At the start: 0 parts

Commit message: Adding all Schematic Element
Parts:
- added BT1: Battery, symbol Device:Battery
- added C1, C2, C3, C4: C, SparkFun-Capacitor:C_0603_1608Metric, symbol SparkFun-Capacitor:C
- added C5: C_Polarized, symbol Device:C_Polarized
- added D1, D2: LED, SparkFun-LED:LED_0603_1608Metric, symbol SparkFun-LED:LED
- added H1, H2, H3, H4: MountingHole, symbol Mechanical:MountingHole
- added R1, R2, R3, R4, R5, R6, R7: R, symbol Device:R
- added U1, U2: 24LC1025, symbol Memory_EEPROM:24LC1025
- added U3: ATmega328P, SparkFun-Semiconductor-Standard:TQFP-32_7x7mm_P0.8mm, symbol SparkFun-IC-Microcontroller:ATmega328P-AU
- added U4: DS1337S_, DS1337S_:SOIC127P600X175-8N, symbol DS1337S_:DS1337S_
- added Y1, Y2: Crystal, symbol Device:Crystal
Connections:
- new net: U3.21 (GND), U3.3 (GND), U3.5 (GND)
- new net: U3.4 (VCC), U3.6 (VCC)
Other:
- added sheet connectors (connectors.kicad_sch)
- title: (none) -> ${project_name}

Commit message: Editing some footprints
Parts:
- BT1: footprint (none) -> TerminalBlock_Phoenix:TerminalBlock_Phoenix_MPT-0,5-2-2.54_1x02_P2.54mm_Horizontal
- C1, C4: value C -> 0.1uF; footprint SparkFun-Capacitor:C_0603_1608Metric -> Capacitor_SMD:C_0805_2012Metric
- C2, C3: value C -> 22pF; footprint SparkFun-Capacitor:C_0603_1608Metric -> Capacitor_SMD:C_0805_2012Metric
- C5: value C_Polarized -> 100nF; footprint (none) -> Capacitor_SMD:C_0805_2012Metric
- D1, D2: footprint SparkFun-LED:LED_0603_1608Metric -> LED_SMD:LED_0805_2012Metric
- H1, H2, H3, H4: footprint (none) -> MountingHole:MountingHole_2.1mm
- R1: value R -> 10K; footprint (none) -> Resistor_SMD:R_0805_2012Metric
- R2, R3: value R -> 4.7k; footprint (none) -> Resistor_SMD:R_0805_2012Metric
- R4, R5: value R -> 10k; footprint (none) -> Resistor_SMD:R_0805_2012Metric
- R6, R7: value R -> 330; footprint (none) -> Resistor_SMD:R_0805_2012Metric
- U1, U2: footprint (none) -> Package_SO:SOIC-8_3.9x4.9mm_P1.27mm
- U3: footprint SparkFun-Semiconductor-Standard:TQFP-32_7x7mm_P0.8mm -> footprints:QFP80P900X900X120-32N
- U4: footprint DS1337S_:SOIC127P600X175-8N -> footprints:SOIC127P600X175-8N
- Y1: value Crystal -> 16MHz; footprint (none) -> Crystal:Crystal_SMD_5032-2Pin_5.0x3.2mm_HandSoldering
- Y2: value Crystal -> 32.768 KHz; footprint (none) -> Crystal:Crystal_SMD_5032-2Pin_5.0x3.2mm_HandSoldering
Other:
- moved on the sheet: BT1, C1, C2, C3, C4, C5, D1, D2, H1, H2, H3, H4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

Commit message: Finishing Wiring
Connections:
- net GND: now reaches R6.1
- net GND: now also BT1.2 (-), C1.1, C2.1, C3.1, C4.2, C5.2, R7.1, U1.4 (GND), U1.7 (WP), U2.2 (A1), U2.4 (GND), U2.7 (WP), U3.21 (GND), U3.3 (GND), U3.5 (GND), U4.4 (GND)
- net at R6.2: now also D2.1 (K)
- net at C3.2: now also U3.8 (XTAL2/PB7), Y1.1
- net VCC: now reaches U1.1 (A0)
- net VCC: now also BT1.1 (+), C1.2, C5.1, D2.2 (A), R1.1, R2.1, R3.1, R4.1, R5.1, U1.2 (A1), U1.3 (A2), U1.8 (VCC), U2.1 (A0), U2.3 (A2), U2.8 (VCC), U3.18 (AVCC), U3.4 (VCC), U3.6 (VCC), U4.8 (VCC)
- net SDA: now reaches U1.5 (SDA)
- net SDA: now also R3.2, U2.5 (SDA), U3.27 (PC4), U4.5 (SDA)
- net SCL: now reaches U1.6 (SCL)
- net SCL: now also D1.2 (A), R2.2, U2.6 (SCL), U3.17 (PB5), U3.28 (PC5), U4.6 (SCL)
- net at U4.1 (X1): now also Y2.2
- net at U4.2 (X2): now also Y2.1
- net at U4.3 (~{INTA}): now also R5.2
- net at U4.7 (SQW/~INT): now also R4.2
- net D3: now reaches U3.1 (PD3)
- net D6: now reaches U3.10 (PD6)
- net D7: now reaches U3.11 (PD7)
- net D8: now reaches U3.12 (PB0)
- net MOSI: now reaches U3.15 (PB3)
- net MISO: now reaches U3.16 (PB4)
- net D4: now reaches U3.2 (PD4)
- net at U3.20 (AREF): now also C4.1
- net RESET: now reaches U3.29 (~{RESET}/PC6)
- net RESET: now also R1.2
- net RX: now reaches U3.30 (PD0)
- net TX: now reaches U3.31 (PD1)
- net D2: now reaches U3.32 (PD2)
- net at U3.7 (XTAL1/PB6): now also C2.2, Y1.2
- net D5: now reaches U3.9 (PD5)
- net at R7.2: now also D1.1 (K)
- no-connect marks 0 -> 8
Other:
- sheet connectors ports: added D2, D3, D4, D5, D6, D7, D8, GND, MISO, MOSI, RESET, RX, SCL, SDA, TX, VCC; removed none
- moved on the sheet: BT1, C1, C2, C3, C4, C5, D1, D2, R1, R2, R4, R5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

Commit message: Components find there home
Parts:
- BT1: footprint TerminalBlock_Phoenix:TerminalBlock_Phoenix_MPT-0,5-2-2.54_1x02_P2.54mm_Horizontal -> Connector_PinHeader_2.54mm:PinHeader_2x01_P2.54mm_Vertical
Changed lines of the file:
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@@
 			)
 		)
-		(property "Footprint" "TerminalBlock_Phoenix:TerminalBlock_Phoenix_MPT-0,5-2-2.54_1x02_P2.54mm_Horizontal"
+		(property "Footprint" "Connector_PinHeader_2.54mm:PinHeader_2x01_P2.54mm_Vertical"
 			(at 192.024 58.42 90)
 			(effects
